File: tp2/sources/ea2_tp2_opamp/ea2_tp2_opamp.kicad_pcb (KiCad board)
At the start: 4 copper layers, 66 x 50.8 mm, 45 parts, among them U1 TL084, U2 TL084, U3 TL082

Commit message: tp2: Metanse la pcb en el orto
Parts:
- moved R10 97.1 mm to (127.0, 86.4)
- moved U3 88.2 mm to (142.2, 106.7)
- moved C1 88.2 mm to (134.6, 91.5)
- moved C4 88.2 mm to (172.7, 91.5)
- moved R11 88.2 mm to (134.6, 119.4)
- moved R12 88.2 mm to (116.8, 119.4)
- moved R18 88.2 mm to (116.8, 96.5)
- moved R2 88.2 mm to (127.0, 81.3)
- moved R21 88.2 mm to (172.7, 119.4)
- moved R25 88.2 mm to (160.0, 109.2)
- moved R26 88.2 mm to (170.2, 109.2)
- moved R27 88.2 mm to (170.2, 86.4)
- moved R28 88.2 mm to (162.6, 109.2)
- moved R29 88.2 mm to (142.2, 109.2)
- moved R30 88.2 mm to (149.9, 86.4)
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Routing:
- net /integrated_pre: track 45.7 -> 26.5 mm
- net +12V: track 81.2 -> 90.7 mm, vias 0 -> 2
- net Net-(U1D-+): track 22.9 -> 16.0 mm
- net 0: track 250.1 -> 256.8 mm
- net /vi_offseted: track 50.8 -> 51.9 mm
- net Net-(R34-Pad1): vias 0 -> 1
Other:
- board size 66 x 50.8 mm -> 68.6 x 53.3 mm
- board text added: "1"
- board text added: "10"
- board text added: "11"
- board text added: "12"
- board text added: "13"
- board text added: "14"
- board text added: "15"
- board text added: "16"
- board text added: "17"
- board text added: "18"
- board text added: "19"
- board text added: "2"
- board text added: "20"
- board text added: "21"
- board text added: "22"
- board text added: "23"
- board text added: "24"
- board text added: "3"
- board text added: "4"
- board text added: "5"
- board text added: "6"
- board text added: "7"
- board text added: "8"
- board text added: "9"
- board text added: "A"
- board text added: "B"
- board text added: "C"
- board text added: "D"
- board text added: "E"
- board text added: "F"
- board text added: "G"
- board text added: "H"
- board text added: "I"
- board text added: "J"
- board text added: "K"
- board text added: "L"
- board text added: "M"
- board text added: "N"
- board text added: "O"
- board text added: "P"
- board text added: "Q"
- board text added: "R"
