File: tp3/pcb/pcb.kicad_pcb (KiCad board)
At the start: 2 copper layers, 49.5 x 33.5 mm, 18 parts, among them J1 Screw_Terminal_01x02, J2 Screw_Terminal_01x03, J3 Conn_01x02_Pin, U1 TL084

Commit message: tp3: Incrusta modelos 3d y corrige pistas pcb
Routing:
- net /V_Processed: track 36.3 -> 34.5 mm
- net +15V: track 55.1 -> 54.1 mm
- net Net-(U1D-+): track 21.4 -> 22.3 mm
- net /V2: track 23.1 -> 22.5 mm

Commit message: fix zone clearance
Parts:
- added G***: LOGO, Samacsys:fucku, F.Cu at (189.2, 85.7)

Commit message: tp3: casi casi terminado falta corregir anexo noma
Parts:
- removed G***: LOGO, Samacsys:fucku
- C1, C2: value 12u -> 2.2u
- C3, C4: value 22n -> 2.2n
- R4, R5, R6, R7: value 100k -> 1M
- R8: value 100k -> 220k
- moved C1 68.5 mm to (91.2, 133.2)
- moved C2 68.5 mm to (93.2, 158.2)
- moved C3 68.5 mm to (117.4, 147.2)
- moved C4 68.5 mm to (117.7, 154.7)
- moved J2 68.5 mm to (127.1, 150.2)
- moved R2 68.5 mm to (83.9, 136.7)
- moved R3 68.5 mm to (83.9, 154.2)
- moved R4 68.5 mm to (97.4, 158.2)
- moved R5 68.5 mm to (97.4, 133.2)
- moved R6 68.5 mm to (110.4, 158.2)
- moved R7 68.5 mm to (110.4, 150.7)
- moved R8 68.5 mm to (120.5, 133.2)
- moved R9 68.5 mm to (120.4, 136.7)
- moved RV1 68.5 mm to (118.5, 142.2)
- moved J1 68.5 mm to (86.9, 147.6)
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