File: tp3/pcb/pcb.kicad_sch (KiCad schematic)
At the start: 18 parts, among them J1 Screw_Terminal_01x02, J2 Screw_Terminal_01x03, J3 Conn_01x02_Pin, U1 TL084

Commit message: Corrige en esquematico no inversor
Connections:
- net V_Processed: now also U1.12 (+); no longer U1.13 (-)
- net at R8.1, R9.2: now also U1.13 (-); no longer U1.12 (+)
Changed lines of the file:
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@@
 		(lib_id "Amplifier_Operational:TL084")
 		(at 208.28 125.73 0)
+		(mirror x)
 		(unit 4)
 		(body_style 1)
@@
 		(dnp no)
 		(property "Reference" "U1"
-			(at 208.28 115.57 0)
+			(at 208.28 135.89 0)
 			(show_name no)
 			(do_not_autoplace no)
@@
 		)
 		(property "Value" "TL084"
-			(at 208.28 118.11 90)
+			(at 208.28 133.35 90)
 			(show_name no)
 			(do_not_autoplace no)
@@
 		)
 		(property "Footprint" "Package_DIP:DIP-14_W7.62mm_Socket_LongPads"
-			(at 207.01 123.19 0)
+			(at 207.01 128.27 0)
 			(hide yes)
 			(show_name no)
@@
 		)
 		(property "Datasheet" "http://www.ti.com/lit/ds/symlink/tl081.pdf"
-			(at 209.55 120.65 0)
+			(at 209.55 130.81 0)
 			(hide yes)
 			(show_name no)

Commit message: Diseña placa V2
Parts:
- added C5, C6: 100 nF, Capacitor_THT:C_Disc_D5.0mm_W2.5mm_P2.50mm, symbol Device:C
Connections:
- net +15V: now also C6.1
- net -15V: now also C5.1
- net GNDREF: now also C5.2, C6.2; no longer J1.2 (Pin_2), U1.3 (+)
- net V_N: now reaches C1.1, R2.2
- net V_N: now also U1.7; no longer U1.1
- net Vi_N: now reaches U1.5 (+)
- net Vi_N: now also J1.2 (Pin_2); no longer J1.1 (Pin_1)
- net at R1.1, R2.1: now also U1.6 (-); no longer U1.2 (-)
- net at R1.2, R3.1: now also U1.2 (-); no longer U1.6 (-)
- net V_P: now reaches C2.2, R3.2
- net V_P: now also U1.1; no longer U1.7
- net V1 renamed Vo_N
- net V2 renamed Vo_P
- new net Vi_P: J1.1 (Pin_1), U1.3 (+)
Other:
- moved on the sheet: U1A, U1B
