File: tp3/pcb/pcb.kicad_sch (KiCad schematic)
At the start: 18 parts, among them J1 Screw_Terminal_01x02, J2 Screw_Terminal_01x03, J3 Conn_01x02_Pin, U1 TL084

Commit message: tp3: casi casi terminado falta corregir anexo noma
Parts:
- C1, C2: value 12u -> 2.2u
- C3, C4: value 22n -> 2.2n
- R1: value 4580 -> 4k7
- R4, R5, R6, R7: value 100k -> 1M
- R8: value 100k -> 220k
Changed lines of the file:
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@@
 			)
 		)
-		(property "Value" "12u"
+		(property "Value" "2.2u"
 			(at 102.87 55.88 90)
 			(show_name no)
@@
 			)
 		)
-		(property "Value" "22n"
+		(property "Value" "2.2n"
 			(at 86.36 147.3199 0)
 			(show_name no)
@@
 			)
 		)
-		(property "Value" "4580"
+		(property "Value" "4k7"
 			(at 81.28 77.4699 0)
 			(show_name no)
@@
 			)
 		)
-		(property "Value" "12u"
+		(property "Value" "2.2u"
 			(at 102.87 86.36 90)
 			(show_name no)
@@
 			)
 		)
-		(property "Value" "100k"
+		(property "Value" "1M"
 			(at 114.3 57.15 90)
 			(show_name no)
@@
 			)
 		)
-		(property "Value" "100k"
+		(property "Value" "220k"
 			(at 208.28 104.14 90)
 			(show_name no)
@@
 			)
 		)
-		(property "Value" "100k"
+		(property "Value" "1M"
 			(at 74.93 147.3199 0)
 			(show_name no)
@@
 			)
 		)
-		(property "Value" "22n"
+		(property "Value" "2.2n"
 			(at 81.28 124.968 90)
 			(show_name no)
@@
 			)
 		)
-		(property "Value" "100k"
+		(property "Value" "1M"
 			(at 81.28 110.49 90)
 			(show_name no)
@@
 			)
 		)
-		(property "Value" "100k"
+		(property "Value" "1M"
 			(at 114.3 87.63 90)
 			(show_name no)
