File: tp3/sources/pcb/pcb.kicad_pcb (KiCad board)
At the start: 2 copper layers, 49.5 x 33.5 mm, 18 parts, among them J1 Screw_Terminal_01x02, J2 Screw_Terminal_01x03, J3 Conn_01x02_Pin, U1 TL084

Commit message: Webada PCB
Parts:
- added C5: 100 nF, Capacitor_THT:C_Disc_D5.0mm_W2.5mm_P2.50mm, F.Cu at (128.8, 121.7)
- added C6: 100 nF, Capacitor_THT:C_Disc_D5.0mm_W2.5mm_P2.50mm, F.Cu at (128.8, 147.1)
- added G***: LOGO, Samacsys:fucku, F.Cu at (189.2, 85.7)
- C1, C2: value 2.2u -> 12u
- C3, C4: value 2.2n -> 22n
- R4, R5, R6, R7: value 1M -> 100k
- R8: value 220k -> 100k
- moved C2 56.4 mm to (128.8, 114.5)
- moved R4 56.4 mm to (132.9, 114.5)
- moved R3 46.8 mm to (120.0, 124.5), turned to 90 degrees
- moved R6 42.5 mm to (150.9, 145.3), turned to 180 degrees
- moved R5 40.1 mm to (132.9, 151.9)
- moved C1 39.8 mm to (126.3, 151.9)
- moved RV1 37.6 mm to (155.2, 133.8), turned to -90 degrees
- moved R2 36.5 mm to (120.0, 141.5), turned to -90 degrees
- moved R7 33.8 mm to (140.4, 135.0)
- moved R8 31.1 mm to (149.5, 122.1)
- moved J3 30.9 mm to (152.3, 118.6)
- moved U1 30.8 mm to (126.7, 125.8)
- moved R9 30.5 mm to (149.9, 128.9)
- moved C3 30.2 mm to (146.7, 140.0)
- moved J2 29.2 mm to (156.3, 151.3)
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Connections:
- net /V1 renamed /Vo_N
- net /V2 renamed /Vo_P
- C1 pad 1: Net-(C1-Pad1) -> /V_N
- C2 pad 2: Net-(C2-Pad2) -> /V_P
- J1 pad 1: Net-(J1-Pin_1) -> /Vi_P
- J1 pad 2: GNDREF -> /Vi_N
- R1 pad 1: Net-(U1A--) -> Net-(U1B--)
- R1 pad 2: Net-(U1B--) -> Net-(U1A--)
- R2 pad 1: Net-(U1A--) -> Net-(U1B--)
- R2 pad 2: Net-(C1-Pad1) -> /V_N
- R3 pad 1: Net-(U1B--) -> Net-(U1A--)
- R3 pad 2: Net-(C2-Pad2) -> /V_P
- R8 pad 1: Net-(U1D-+) -> Net-(U1D--)
- R9 pad 2: Net-(U1D-+) -> Net-(U1D--)
- U1 pad 1: Net-(C1-Pad1) -> /V_P
- U1 pad 12: Net-(U1D-+) -> /V_Processed
- U1 pad 13: /V_Processed -> Net-(U1D--)
- U1 pad 3: GNDREF -> /Vi_P
- U1 pad 5: Net-(J1-Pin_1) -> /Vi_N
- U1 pad 7: Net-(C2-Pad2) -> /V_N
Routing:
- net -15V: track 23.2 -> 76.1 mm
- net Net-(U1D--): track 0.00 -> 22.9 mm, vias 0 -> 2
- net Net-(U1D-+): track 22.3 -> 0.00 mm
- net /V_N: track 0.00 -> 19.2 mm
- net /V_P: track 0.00 -> 17.9 mm
- net /Vi_N: track 0.00 -> 17.8 mm
- net /Vi_P: track 0.00 -> 17.7 mm
- net /Vo_P: track 22.5 -> 36.0 mm
- net Net-(J1-Pin_1): track 12.2 -> 0.00 mm
- net Net-(C2-Pad2): track 11.3 -> 0.00 mm
- net Net-(C1-Pad1): track 11.3 -> 0.00 mm
- net /V_Processed: track 34.5 -> 26.0 mm, vias 4 -> 2
- net /Vo_N: track 46.4 -> 39.3 mm
- net Net-(U1B--): track 16.8 -> 10.3 mm
- net Net-(U1A--): track 16.6 -> 10.3 mm
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Other:
- board size 49.5 x 33.5 mm -> 55.5 x 50 mm
