File: tp3/sources/pcb/pcb.kicad_sch (KiCad schematic)
At the start: 18 parts, among them J1 Screw_Terminal_01x02, J2 Screw_Terminal_01x03, J3 Conn_01x02_Pin, U1 TL084

Commit message: Webada PCB
Parts:
- added C5, C6: 100 nF, Capacitor_THT:C_Disc_D5.0mm_W2.5mm_P2.50mm, symbol Device:C
- C1, C2: value 2.2u -> 12u
- C3, C4: value 2.2n -> 22n
- R1: value 4k7 -> 4580
- R4, R5, R6, R7: value 1M -> 100k
- R8: value 220k -> 100k
Connections:
- net +15V: now also C6.1
- net -15V: now also C5.1
- net GNDREF: now also C5.2, C6.2; no longer J1.2 (Pin_2), U1.3 (+)
- net V_Processed: now also U1.12 (+); no longer U1.13 (-)
- net V_N: now reaches C1.1, R2.2
- net V_N: now also U1.7; no longer U1.1
- net Vi_N: now reaches U1.5 (+)
- net Vi_N: now also J1.2 (Pin_2); no longer J1.1 (Pin_1)
- net at R1.1, R2.1: now also U1.6 (-); no longer U1.2 (-)
- net at R1.2, R3.1: now also U1.2 (-); no longer U1.6 (-)
- net V_P: now reaches C2.2, R3.2
- net V_P: now also U1.1; no longer U1.7
- net at R8.1, R9.2: now also U1.13 (-); no longer U1.12 (+)
- net V1 renamed Vo_N
- net V2 renamed Vo_P
- new net Vi_P: J1.1 (Pin_1), U1.3 (+)
Other:
- moved on the sheet: U1A, U1B
