File: tp4/sources/ampli.kicadproj/3band_eq.kicad_sch (KiCad schematic)
At the start: 30 parts, among them U301 TL084, U302 TL084

Commit message: tp4: Agrega pcb y actualiza simulaciones
Parts:
- removed JP301: SolderJumper_3_Open, symbol Jumper:SolderJumper_3_Open
- added C302, C304, C307, C308: 100n, Capacitor_THT:C_Disc_D5.0mm_W2.5mm_P2.50mm, symbol Device:C
- C301: footprint (none) -> Capacitor_THT:C_Rect_L7.2mm_W2.5mm_P5.00mm
- C303: renamed from C302; footprint (none) -> Capacitor_THT:C_Rect_L7.2mm_W2.5mm_P5.00mm
- C305: renamed from C303; footprint (none) -> Capacitor_THT:C_Rect_L7.2mm_W2.5mm_P5.00mm
- C306: renamed from C304; footprint (none) -> Capacitor_THT:C_Rect_L7.2mm_W2.5mm_P5.00mm
- C309: renamed from C305; footprint (none) -> Capacitor_THT:C_Rect_L7.2mm_W2.5mm_P5.00mm
- C310: renamed from C306; footprint (none) -> Capacitor_THT:C_Rect_L7.2mm_W2.5mm_P5.00mm
- C311: renamed from C307; footprint (none) -> Capacitor_THT:C_Rect_L7.2mm_W2.5mm_P5.00mm
- C312: renamed from C308; footprint (none) -> Capacitor_THT:C_Rect_L7.2mm_W2.5mm_P5.00mm
- R301, R302, R303, R304, R305, R306, R307, R308, R309, R310, R311, R312, R313, R314, R315, R316: footprint (none) -> Resistor_THT:R_Axial_DIN0207_L6.3mm_D2.5mm_P10.16mm_Horizontal
- RV301, RV302, RV303: footprint Package_SO:TSSOP-20_4.4x6.5mm_P0.65mm -> Potentiometer_THT:Potentiometer_Omeg_PC16BU_Vertical
- U301, U302: footprint Package_DFN_QFN:Texas_DSQ0010A_WSON-10-1EP_2x2mm_P0.4mm_EP0.9x1.5mm -> Package_DIP:DIP-14_W7.62mm_Socket_LongPads
Connections:
- net +15V: now also C302.1, C308.1
- net -15V: now also C304.2, C307.2
- net GND: now also C302.2, C304.1, C307.1, C308.2
- net V_{i buffered}: now also U301.1, U301.2 (-)
- net V_{ia}: no longer names the net of U301.6 (-)
- net V_{ib}: no longer names the net of U301.5 (+)
- no-connect marks 0 -> 3
