File: tp4/sources/ampli.kicadproj/ampli.kicad_pcb (KiCad board)
At the start: 2 copper layers, 117.1 x 84.6 mm, 66 parts, among them J101 P_POW, J102 AUDIO_IN, J103 N_POW, J104 P_POW, J105 AUDIO_OUT, J106 N_POW, J107 P_POW, J108 AUDIO_IN, J109 N_POW, J110 AUDIO_OUT, Q201 BC337, Q202 BC337, Q203 BC327, Q204 BC327, Q205 BC337, Q206 TIP122, Q207 TIP127, U201 TL082, U301 TL084, U302 TL084

Commit message: tp4: Correcciones finales del esquematico para P=10W
Parts:
- R206: value 12k -> 6k8
Routing:
- net (no net): track 0.00 -> 16.6 mm
- net /Amplificador/GND: track 108.0 -> 97.8 mm
- net /Ecualizador/GND: track 170.4 -> 164.0 mm
